Commit message: 260516

File: Dynamixel/dynamixel_control/poppy_description/robots/Poppy_Humanoid.URDF (robot description, URDF)
Before this commit: robot Poppy_Humanoid, 26 links, 25 joints
Links:
- added link l_wrist
- added link r_wrist
Joints:
- added joint l_wrist_fixed: type fixed, parent l_forearm, child l_wrist, origin xyz=0 0.120 0 rpy=0 0 0
- added joint r_wrist_fixed: type fixed, parent r_forearm, child r_wrist, origin xyz=0 0.120 0 rpy=0 0 0
